Commit message: attempted autonomous driving and tried to fix errors

File: src/my_robot_description/urdf/my_robot.urdf.xacro (robot description, xacro)
@@ -1,111 +1,158 @@
 <?xml version="1.0"?>
-<robot xmlns:xacro="http://www.ros.org/wiki/xacro" name="my_robot">
-    <!-- RViz2 için Renk Tanımları -->
+<robot xmlns:xacro="http://www.ros.org/wiki/xacro" name="teknofest_agv">
+    <!-- RViz2 Renkleri -->
     <material name="blue"><color rgba="0.1 0.2 0.8 1"/></material>
     <material name="black"><color rgba="0.1 0.1 0.1 1"/></material>
     <material name="white"><color rgba="0.9 0.9 0.9 1"/></material>
-    <!-- 1. KÖK NOKTA (KDL uyarısını önleyen ağırlıksız yer izdüşümü) -->
-    <link name="base_footprint"/>
-    <!-- base_footprint ile base_link arasındaki sabit bağlantı (Gövdeyi yerden 8cm yukarıda tutar) -->
-    <joint name="base_joint" type="fixed">
-        <parent link="base_footprint"/>
-        <child link="base_link"/>
-        <origin xyz="0 0 0.08" rpy="0 0 0"/>
-    </joint>
-    <!-- 2. ANA GÖVDE (Şasi) -->
+    <material name="red"><color rgba="0.8 0.1 0.1 1"/></material>
+    <!-- 1. ANA GÖVDE (Doğrudan base_link - TF karmaşasını sıfırlar) -->
     <link name="base_link">
         <visual>
-            <geometry><box size="0.5 0.3 0.1"/></geometry>
+            <geometry><box size="0.5 0.4 0.2"/></geometry>
             <material name="blue"/>
         </visual>
         <collision>
-            <geometry><box size="0.5 0.3 0.1"/></geometry>
+            <geometry><box size="0.5 0.4 0.2"/></geometry>
         </collision>
         <inertial>
-            <mass value="2.0"/>
-            <inertia ixx="0.02" ixy="0" ixz="0" iyy="0.04" iyz="0" izz="0.05"/>
+            <mass value="10.0"/>
+            <inertia ixx="0.1" ixy="0" ixz="0" iyy="0.1" iyz="0" izz="0.1"/>
         </inertial>
     </link>
-    <!-- 3. TEKERLEK MAKROSU (Fonksiyon gibi: İsim ve Y-konumu alır, tekerleği üretir) -->
-    <xacro:macro name="drive_wheel" params="prefix y_reflect">
-        <link name="${prefix}_wheel">
-            <visual>
-                <!-- Silindiri dikeyden yataya (tekerlek pozisyonuna) çevirmek için X ekseninde 90 derece (pi/2) döndürüyoruz -->
-                <origin xyz="0 0 0" rpy="${-pi/2} 0 0"/>
-                <geometry><cylinder radius="0.06" length="0.04"/></geometry>
-                <material name="black"/>
-            </visual>
-            <collision>
-                <origin xyz="0 0 0" rpy="${-pi/2} 0 0"/>
-                <geometry><cylinder radius="0.06" length="0.04"/></geometry>
-            </collision>
-            <inertial>
-                <origin xyz="0 0 0" rpy="${-pi/2} 0 0"/>
-                <mass value="0.3"/>
-                <inertia ixx="0.0003" ixy="0" ixz="0" iyy="0.0003" iyz="0" izz="0.0005"/>
-            </inertial>
-        </link>
-        <!-- Continuous Joint: Sınır olmadan 360 derece dönebilen motorlu tekerlek eklemi -->
-        <joint name="${prefix}_wheel_joint" type="continuous">
-            <parent link="base_link"/>
-            <child link="${prefix}_wheel"/>
-            <origin xyz="-0.15 ${y_reflect * 0.17} -0.02" rpy="0 0 0"/>
-            <axis xyz="0 1 0"/> <!-- Y ekseni etrafında döner -->
-        </joint>
-        <gazebo reference="${prefix}_wheel">
-            <material>Gazebo/Black</material>
-        </gazebo>
-    </xacro:macro>
-    <!-- Makroyu çağırarak Sol ve Sağ tekerlekleri oluşturuyoruz -->
-    <xacro:drive_wheel prefix="left" y_reflect="1"/>
-    <xacro:drive_wheel prefix="right" y_reflect="-1"/>
-    <!-- 4. ÖN DENGE TEKERLEĞİ (Caster Wheel - Küre şeklinde) -->
-    <link name="caster_wheel">
+    <gazebo reference="base_link"><material>Gazebo/Blue</material></gazebo>
+    <!-- 2. SAĞ TEKERLEK -->
+    <link name="sag_tekerlek">
         <visual>
-            <geometry><sphere radius="0.03"/></geometry>
+            <geometry><cylinder radius="0.1" length="0.05"/></geometry>
+            <material name="black"/>
+        </visual>
+        <collision>
+            <geometry><cylinder radius="0.1" length="0.05"/></geometry>
+        </collision>
+        <inertial>
+            <mass value="1.0"/>
+            <inertia ixx="0.01" ixy="0" ixz="0" iyy="0.01" iyz="0" izz="0.01"/>
+        </inertial>
+    </link>
+    <gazebo reference="sag_tekerlek">
+        <material>Gazebo/Black</material>
+        <mu1>1.0</mu1><mu2>1.0</mu2><kp>1000000.0</kp><kd>100.0</kd>
+    </gazebo>
+    <joint name="sag_teker_mafsali" type="continuous">
+        <parent link="base_link"/>
+        <child link="sag_tekerlek"/>
+        <origin xyz="0.15 -0.225 -0.1" rpy="1.5708 0 0"/>
+        <axis xyz="0 0 -1"/>
+    </joint>
+    <!-- 3. SOL TEKERLEK -->
+    <link name="sol_tekerlek">
+        <visual>
+            <geometry><cylinder radius="0.1" length="0.05"/></geometry>
+            <material name="black"/>
+        </visual>
+        <collision>
+            <geometry><cylinder radius="0.1" length="0.05"/></geometry>
+        </collision>
+        <inertial>
+            <mass value="1.0"/>
+            <inertia ixx="0.01" ixy="0" ixz="0" iyy="0.01" iyz="0" izz="0.01"/>
+        </inertial>
+    </link>
+    <gazebo reference="sol_tekerlek">
+        <material>Gazebo/Black</material>
+        <mu1>1.0</mu1><mu2>1.0</mu2><kp>1000000.0</kp><kd>100.0</kd>
+    </gazebo>
+    <joint name="sol_teker_mafsali" type="continuous">
+        <parent link="base_link"/>
+        <child link="sol_tekerlek"/>
+        <origin xyz="0.15 0.225 -0.1" rpy="1.5708 0 0"/>
+        <axis xyz="0 0 -1"/>
+    </joint>
+    <!-- 4. ÖN SARHOŞ (CASTER) TEKERLEK -->
+    <link name="sarhos_tekerlek">
+        <visual>
+            <geometry><sphere radius="0.05"/></geometry>
             <material name="white"/>
         </visual>
         <collision>
-            <geometry><sphere radius="0.03"/></geometry>
+            <geometry><sphere radius="0.05"/></geometry>
         </collision>
         <inertial>
-            <mass value="0.1"/>
-            <inertia ixx="0.0001" ixy="0" ixz="0" iyy="0.0001" iyz="0" izz="0.0001"/>
+            <mass value="0.5"/>
+            <inertia ixx="0.01" ixy="0" ixz="0" iyy="0.01" iyz="0" izz="0.01"/>
         </inertial>
     </link>
-    <joint name="caster_wheel_joint" type="fixed">
+    <gazebo reference="sarhos_tekerlek">
+        <material>Gazebo/White</material>
+        <mu1>0.0</mu1><mu2>0.0</mu2>
+    </gazebo>
+    <joint name="sarhos_mafsal" type="fixed">
         <parent link="base_link"/>
-        <child link="caster_wheel"/>
-        <origin xyz="0.15 0 -0.05" rpy="0 0 0"/>
+        <child link="sarhos_tekerlek"/>
+        <origin xyz="-0.2 0 -0.15" rpy="0 0 0"/>
     </joint>
-    <!-- 5. GAZEBO RENK VE FİZİK AYARLARI -->
-    <gazebo reference="base_link">
-        <material>Gazebo/Blue</material>
+    <!-- 5. LIDAR SENSÖRÜ (Eski kararlı 0 - 6.28 tarama açısı) -->
+    <link name="lidar_link">
+        <visual>
+            <geometry><cylinder radius="0.05" length="0.04"/></geometry>
+            <material name="red"/>
+        </visual>
+        <collision>
+            <geometry><cylinder radius="0.05" length="0.04"/></geometry>
+        </collision>
+        <inertial>
+            <mass value="0.2"/>
+            <inertia ixx="0.001" ixy="0" ixz="0" iyy="0.001" iyz="0" izz="0.001"/>
+        </inertial>
+    </link>
+    <gazebo reference="lidar_link"><material>Gazebo/Red</material></gazebo>
+    <joint name="lidar_mafsali" type="fixed">
+        <parent link="base_link"/>
+        <child link="lidar_link"/>
+        <origin xyz="0 0 0.12" rpy="0 0 0"/>
+    </joint>
+    <gazebo reference="lidar_link">
+        <sensor name="rplidar_a2" type="ray">
+            <always_on>true</always_on>
+            <visualize>true</visualize>
+            <update_rate>10</update_rate>
+            <ray>
+                <scan>
+                    <horizontal>
+                        <samples>360</samples>
+                        <resolution>1.0</resolution>
+                        <min_angle>0.0</min_angle>
+                        <max_angle>6.28</max_angle>
+                    </horizontal>
+                </scan>
+                <range>
+                    <min>0.15</min>
+                    <max>12.0</max>
+                    <resolution>0.01</resolution>
+                </range>
+            </ray>
+            <plugin name="lidar_controller" filename="libgazebo_ros_ray_sensor.so">
+                <ros><remapping>~/out:=scan</remapping></ros>
+                <output_type>sensor_msgs/LaserScan</output_type>
+                <frame_name>lidar_link</frame_name>
+            </plugin>
+        </sensor>
     </gazebo>
-    <gazebo reference="caster_wheel">
-        <material>Gazebo/White</material>
-        <!-- Ön küre tekerleğin zeminde yağ gibi kayması için sürtünmeyi (mu1, mu2) sıfıra yaklaştırıyoruz -->
-        <mu1 value="0.001"/>
-        <mu2 value="0.001"/>
-    </gazebo>
-    <!-- 6. GAZEBO DİFERANSİYEL SÜRÜŞ EKLENTİSİ (Motor Kontrolcüsü) -->
+    <!-- 6. DİFERANSİYEL SÜRÜŞ EKLENTİSİ (base_link referanslı stabil TF) -->
     <gazebo>
         <plugin name="diff_drive" filename="libgazebo_ros_diff_drive.so">
-            <left_joint>left_wheel_joint</left_joint>
-            <right_joint>right_wheel_joint</right_joint>
-            <!-- İki tekerlek arası mesafe (0.17 * 2 = 0.34m) ve tekerlek çapı (0.06 * 2 = 0.12m) -->
-            <wheel_separation>0.34</wheel_separation>
-            <wheel_diameter>0.12</wheel_diameter>
+            <left_joint>sol_teker_mafsali</left_joint>
+            <right_joint>sag_teker_mafsali</right_joint>
+            <wheel_separation>0.45</wheel_separation>
+            <wheel_diameter>0.2</wheel_diameter>
             <max_wheel_torque>20</max_wheel_torque>
             <max_wheel_acceleration>1.0</max_wheel_acceleration>
-            <!-- Odometri (konum hesabı) ve koordinat dönüşümlerini (TF) yayınla -->
-            <odometry_frame>odom</odometry_frame>
-            <robot_base_frame>base_footprint</robot_base_frame>
             <publish_odom>true</publish_odom>
             <publish_odom_tf>true</publish_odom_tf>
             <publish_wheel_tf>true</publish_wheel_tf>
+            <command_topic>cmd_vel</command_topic>
+            <odometry_frame>odom</odometry_frame>
+            <robot_base_frame>base_link</robot_base_frame>
         </plugin>
     </gazebo>
-<!-- LIDAR Sensör Modülünü Dahil Et -->
-    <xacro:include filename="$(find my_robot_description)/urdf/lidar.xacro" />
 </robot>
